Commit message: Fixed model and buoyancy issues

File: bluerov2_description/urdf/base.xacro (robot description, xacro)
@@ -2,5 +2,5 @@
 <robot xmlns:xacro="http://www.ros.org/wiki/xacro">
   <!-- Loading some constants -->
-  <xacro:include filename="$(find uuv_descriptions)/models/common/urdf/common.urdf.xacro"/>
+  <xacro:include filename="$(find uuv_descriptions)/urdf/common.urdf.xacro"/>
   <!-- Loading file with sensor macros -->
   <xacro:include filename="$(find uuv_sensor_ros_plugins)/urdf/sensor_snippets.xacro"/>
@@ -72,10 +72,10 @@
         </visual>
         <!-- In rexrov2_base they made collision planes to minize the GPU load -->
-        <!-- <collision>
+        <collision>
           <origin xyz="0 0 0" rpy="0 0 0"/>
           <geometry>
             <mesh filename="${collision_mesh_file}" scale="1 1 1" />
           </geometry>
-        </collision> -->
+        </collision>
       </link>
     <gazebo reference="${namespace}/base_link">

File: bluerov2_description/urdf/sensors.xacro (robot description, xacro)
@@ -18,10 +18,10 @@
   </xacro:default_pressure>
   <!-- Beacon Sensor  -->
-  <xacro:default_beacon namespace="${namespace}" parent_link="${namespace}/base_link">
+  <!-- <xacro:default_beacon namespace="${namespace}" parent_link="${namespace}/base_link">
     <origin xyz="0 0 0" rpy="0 0 0"/>
-  </xacro:default_beacon>
+  </xacro:default_beacon> -->
   <!-- Mount a camera -->
-  <!-- <xacro:default_camera namespace="${namespace}" parent_link="${namespace}/base_link" suffix="front">
+  <xacro:default_camera namespace="${namespace}" parent_link="${namespace}/base_link" suffix="front">
     <origin xyz="0 0 0.2" rpy="0 0 0"/>
-  </xacro:default_camera> -->
+  </xacro:default_camera>
 </robot>

Commit message: Balancing BlueROV2

File: bluerov2_description/urdf/base.xacro (robot description, xacro)
@@ -13,5 +13,5 @@
   -->
   <!-- Mass -->
-  <xacro:property name="mass" value="10"/>
+  <xacro:property name="mass" value="11.15"/>
   <!-- Describing the dimensions of the vehicle's bounding box: width, length, height -->
   <xacro:property name="x_size" value="0.448"/>
@@ -28,5 +28,5 @@
   assume NWU (otherwise cob is below cog?). 0.155
   -->
-  <xacro:property name="cob" value="0 0 0"/>
+  <xacro:property name="cob" value="0 0 0.15"/>
   <!-- Fluid density -->
   <xacro:property name="rho" value="1028"/>
