Commit message: separated robot descriptions

File: bluerov2_description/robots/bluerov2_rlearning.xacro (robot description, xacro)
@@ -30,5 +30,3 @@
   <!-- Joint state publisher plugin -->
   <xacro:default_joint_state_publisher namespace="$(arg namespace)" update_rate="10"/>
-  <!-- Mount a Pose 3D sensor. -->
-  <xacro:default_pose_3d namespace="bluerov2" parent_link="bluerov2/base_link" />
 </robot>

File: bluerov2_description/urdf/base.xacro (robot description, xacro)
@@ -42,4 +42,5 @@
   regarding the computation of collision forces) -->
   <xacro:property name="collision_mesh_file" value="file://$(find bluerov2_description)/meshes/bluerov2_noprop.stl"/>
+  <xacro:property name="use_simplified_mesh" value="false"/>
   <!-- Vehicle macro -->
   <!-- <xacro:macro name="bluerov2_base" params="namespace debug *gazebo"> -->

File: bluerov2_description/urdf/sensors.xacro (robot description, xacro)
@@ -8,5 +8,5 @@
   -->
   <!-- Mount a Pose 3D sensor. -->
-  <xacro:default_pose_3d namespace="${namespace}" parent_link="${namespace}/base_link" />
+  <!-- <xacro:default_pose_3d namespace="${namespace}" parent_link="${namespace}/base_link" /> -->
   <!-- IMU Sensor -->
   <xacro:default_imu namespace="${namespace}" parent_link="${namespace}/base_link">
@@ -22,6 +22,52 @@
   </xacro:default_beacon> -->
   <!-- Mount a camera -->
-  <xacro:default_camera namespace="${namespace}" parent_link="${namespace}/base_link" suffix="front">
+  <!-- <xacro:default_camera namespace="${namespace}" parent_link="${namespace}/base_link" suffix="front">
     <origin xyz="0 0 0.2" rpy="0 0 0"/>
-  </xacro:default_camera>
+  </xacro:default_camera> -->
+  <link name="bluerov2/camera_link">
+    <inertial>
+      <mass value=".01"/>
+      <inertia ixx="1.0" ixy="0.0" ixz="0.0" iyy="1.0" iyz="0.0" izz="1.0"/>
+    </inertial>
+  </link>
+  <joint name="bluerov2_camera" type="fixed">
+    <parent link="bluerov2/base_link"/>
+    <child link="bluerov2/camera_link"/>
+    <origin xyz=".1 0 -.1" rpy="-1.57 0 -1.57"/>
+  </joint>
+  <gazebo reference="bluerov2/base_link">
+    <sensor type="camera" name="camera_out">
+      <update_rate>30.0</update_rate>
+      <camera name="head">
+        <!-- <pose>4 -4 2 0.0 0.275643 2.356190</pose> -->
+        <pose>.1 0 -.1 0 0 0</pose>
+        <view_controller>orbit</view_controller>
+        <horizontal_fov>1.3962634</horizontal_fov>
+        <image>
+          <width>800</width>
+          <height>600</height>
+          <format>R8G8B8</format>
+        </image>
+        <clip>
+          <near>0.02</near>
+          <far>300</far>
+        </clip>
+      </camera>
+      <plugin name="camera_controller" filename="libCameraBboxPlugin.so">
+      <!-- <plugin name="camera_controller" filename="libcamera_bbox.so"> -->
+        <alwaysOn>true</alwaysOn>
+        <updateRate>0.0</updateRate>
+        <cameraName>camera_out</cameraName>
+        <imageTopicName>image_raw</imageTopicName>
+        <cameraInfoTopicName>camera_info</cameraInfoTopicName>
+        <frameName>camera_link</frameName>
+        <hackBaseline>0.07</hackBaseline>
+        <distortionK1>0.0</distortionK1>
+        <distortionK2>0.0</distortionK2>
+        <distortionK3>0.0</distortionK3>
+        <distortionT1>0.0</distortionT1>
+        <distortionT2>0.0</distortionT2>
+      </plugin>
+    </sensor>
+  </gazebo>
 </robot>
